File: hardware/electrical/display_breakout/display_breakout.kicad_pcb (KiCad board)
At the start: 2 copper layers, 126 x 62.5 mm, 10 parts, among them J1 Conn_02x10_Odd_Even, J2 Conn_01x14_Socket, SW1 RotaryEncoder_Switch, SW2 SW_Push, SW3 SW_Push

Commit message: updated schematic for display_breakout
Parts:
- added C1: 100nF, Capacitor_SMD:C_0603_1608Metric, F.Cu at (204.5, 94.8)
- added C2: 100nF, Capacitor_SMD:C_0603_1608Metric, F.Cu at (204.5, 97.3)
- added C3: 100nF, Capacitor_SMD:C_0603_1608Metric, F.Cu at (204.5, 99.8)
- added C4: 100nF, Capacitor_SMD:C_0603_1608Metric, F.Cu at (204.5, 102.3)
- added C5: 100nF, Capacitor_SMD:C_0603_1608Metric, F.Cu at (204.5, 104.8)
- added Q1: 2N7002, Package_TO_SOT_SMD:SOT-23, F.Cu at (215.0, 67.0)
- added R2: 10k, Resistor_SMD:R_01005_0402Metric, F.Cu at (207.6, 94.3)
- added R3: 10k, Resistor_SMD:R_01005_0402Metric, F.Cu at (207.6, 96.0)
- added R4: 10k, Resistor_SMD:R_01005_0402Metric, F.Cu at (207.6, 97.6)
- added R5: 10k, Resistor_SMD:R_01005_0402Metric, F.Cu at (207.6, 99.3)
- added R6: 10k, Resistor_SMD:R_01005_0402Metric, F.Cu at (207.6, 100.9)
- added R7: 10k, Resistor_SMD:R_01005_0402Metric, F.Cu at (207.6, 102.6)
Connections:
- BZ1 pad 2: GND -> Net-(BZ1--)

Commit message: added display_breakout_small
Connections:
- J2 pad 2: /TOUCH_DO -> /SPI_MISO
- J2 pad 3: /TOUCH_DIN -> /SPI_MOSI
- J2 pad 5: /TOUCH_CLK -> /SPI_CLK
Changed lines of the file:
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@@
 			(layers "*.Cu" "*.Mask")
 			(remove_unused_layers no)
-			(net "/TOUCH_DO")
+			(net "/SPI_MISO")
 			(pinfunction "Pin_2_2")
 			(pintype "passive")
@@
 			(layers "*.Cu" "*.Mask")
 			(remove_unused_layers no)
-			(net "/TOUCH_DIN")
+			(net "/SPI_MOSI")
 			(pinfunction "Pin_3_3")
 			(pintype "passive")
@@
 			(layers "*.Cu" "*.Mask")
 			(remove_unused_layers no)
-			(net "/TOUCH_CLK")
+			(net "/SPI_CLK")
 			(pinfunction "Pin_5_5")
 			(pintype "passive")
