File: hardware/electrical/embo kicad file/embo.kicad_sch (KiCad schematic)
At the start: 97 parts, among them IC1 OPA2354, IC2 OPA2354, J1 Conn_Coaxial, J10 Conn_01x08, J11 Conn_01x08, J12 Conn_01x08, J13 USB_C_Receptacle_USB2.0_16P, J14 24 V PSU input, J15 Conn_01x08, J2 Conn_Coaxial, J3 UART to RPi, J4 JSTXH 6pin Socket 1, J5 JSTXH 6pin Socket 2, J6 motor 1, J7 motor 2, J8 LED Panel, J9 Conn_02x10_Odd_Even, Q1 AO4407A, U1 ESP32-S3-WROOM-1, U2 LM2596S-5, U3 AMS1117-3.3, U4 AD9833xRM

Commit message: PCB trace routing update 50%
Other:
- note added: "01/07/2026"
- note added: "v2.5"
- note removed: "29/06/2026"
- note removed: "v2.2"
Changed lines of the file:
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@@
 		)
 	)
-	(text "v2.2"
+	(text "v2.5"
 		(exclude_from_sim no)
 		(at 343.154 199.136 0)
@@
 		)
 	)
-	(text "29/06/2026"
+	(text "01/07/2026"
 		(exclude_from_sim no)
 		(at 279.908 199.136 0)
@@
 		(lib_id "Device:R")
 		(at 270.51 29.21 0)
+		(mirror y)
 		(unit 1)
 		(body_style 1)
@@
 		(dnp no)
 		(property "Reference" "R38"
-			(at 273.05 27.9399 0)
+			(at 267.97 27.9399 0)
 			(hide yes)
 			(show_name no)
@@
 		)
 		(property "Footprint" "Resistor_SMD:R_0402_1005Metric_Pad0.72x0.64mm_HandSolder"
-			(at 268.732 29.21 90)
+			(at 272.288 29.21 90)
 			(hide yes)
 			(show_name no)

Commit message: fix LM2596S-5 Buck Converter Footprint pinout mismatch and reroute buck converter block to minimise switching circuit loop area
Parts:
- removed C29, C40: 100nF X7R, Capacitor_SMD:C_0402_1005Metric_Pad0.74x0.62mm_HandSolder, symbol Device:C
- removed C32: 10µF X5R 0805, Capacitor_SMD:C_0805_2012Metric, symbol Device:C
Connections:
- net +5V: now also U2.2 (FB); no longer U2.4 (FB)
- net at D4.1 (K), L1.2, Rsnub1.1: now also U2.4 (OUT); no longer U2.2 (OUT)
Other:
- note removed: "VDD3P3 pin 2"
