File: hardware/electrical/embo kicad file/embo.kicad_pcb (KiCad board)
At the start: 4 copper layers, 96.4 x 48.3 mm, 98 parts, among them IC1 OPA2354, IC2 OPA2354, J1 Conn_Coaxial, J10 Conn_01x08, J11 Conn_01x08, J12 Conn_01x08, J13 USB_C_Receptacle_USB2.0_16P, J14 24 V PSU input, J15 Conn_01x08, J2 Conn_Coaxial, J3 UART to RPi, J4 JSTXH 6pin Socket 1, J5 JSTXH 6pin Socket 2, J6 motor 1, J7 motor 2, J8 LED Panel, J9 Conn_02x10_Odd_Even, Q1 AO4407A, U1 ESP32-S3-WROOM-1, U2 LM2596S-5, U3 AMS1117-3.3, U4 AD9833xRM

Commit message: finish routing main PCB
Parts:
- moved C17 0.51 mm to (163.3, 80.3)
- moved C18 0.51 mm to (166.7, 80.3)
Routing:
- net /M2_STEP: track 13.6 -> 103.1 mm, vias 0 -> 5
- net /M2_DIR: track 17.1 -> 98.4 mm, vias 0 -> 2
- net /M2_EN: track 3.54 -> 84.0 mm, vias 0 -> 2
- net /M1_DIR: track 0.00 -> 77.3 mm, vias 0 -> 1
- net /M1_EN: track 3.26 -> 80.1 mm, vias 0 -> 3
- net /M1_STEP: track 0.00 -> 76.7 mm, vias 0 -> 1
- net Net-(J10-Pin_4): track 129.3 -> 137.3 mm
- net /EC11_B (DT): track 46.2 -> 48.9 mm
- net /EC11_SW: track 40.7 -> 43.1 mm
- net /EC11_A (CLK): track 48.9 -> 50.0 mm, vias 0 -> 1
- net Net-(J13-CC1): track 28.1 -> 29.2 mm
- net /TFT_CS: track 42.4 -> 43.5 mm
- net /LIMIT_M2: track 22.2 -> 21.2 mm
- net /LIMIT_M1: track 22.2 -> 21.7 mm
- net GND: track 116.1 -> 115.6 mm, vias 223 -> 250

Commit message: main PCB DRC round 1
Routing:
- net Net-(J13-CC1): track 29.2 -> 10.7 mm, vias 0 -> 2
- net Net-(J10-Pin_4): track 137.3 -> 126.7 mm
- net GND: track 115.6 -> 117.6 mm, vias 250 -> 258
- net +5V: vias 0 -> 4
Other:
- board text added: "30.007 G3"

Commit message: main PCB finishing done
Routing:
- net +3V3: track 44.6 -> 40.2 mm
- net GND: track 117.6 -> 114.0 mm, vias 258 -> 261
- net /M1_EN: track 80.1 -> 79.1 mm, vias 3 -> 2
Other:
- board text added: "30.007 2026"
- board text added: "by Team A&C"
- board text removed: "30.007 G3"
